Commit message: changed cad model for simplified dof

File: src/model/robot.urdf (robot description, URDF)
Before this commit: robot onshape, 21 links, 20 joints
Links:
- removed link leftpivot
- removed link leftpivot_2
- removed link leftservoattachment
- removed link leftservoattachment_2
- removed link rightpivot
- removed link rightpivot_2
- removed link rightservoattachment
- removed link rightservoattachment_2
- added link leftfemur, mass 0.0012188090534078449383; collision mesh filename=package:///bearing_5x8x2.5_v1.stl; collision mesh filename=package:///bearing_5x8x2.5_v1.stl
- added link leftfemur_2, mass 0.0012188090534078449383; collision mesh filename=package:///bearing_5x8x2.5_v1.stl; collision mesh filename=package:///bearing_5x8x2.5_v1.stl
- added link leftfemur_3, mass 0.0012188090534078449383; collision mesh filename=package:///bearing_5x8x2.5_v1.stl; collision mesh filename=package:///bearing_5x8x2.5_v1.stl
- added link leftfemur_4, mass 0.0012188090534078449383; collision mesh filename=package:///bearing_5x8x2.5_v1.stl; collision mesh filename=package:///bearing_5x8x2.5_v1.stl
- link lefthip: mass 0.032471851625270664599 -> 0.035898853366757597916; geometry collision mesh filename=package:///18g_thigh_servo_attachment_v3.stl; collision mesh filename=package:///9g_servo_arm_v1.stl
- link lefthip_2: mass 0.032471851625270671537 -> 0.035898853366757604855; geometry collision mesh filename=package:///18g_thigh_servo_attachment_v3.stl; collision mesh filename=package:///9g_servo_arm_v1.stl
- link rightfoot: mass 0.0052504289083666255342 -> 0.0052504289083666246668
- link rightfoot_2: mass 0.0052504289083666255342 -> 0.0052504289083666246668
- link righthip: mass 0.031925376082855685955 -> 0.035352377824358502401; geometry collision mesh filename=package:///18g_thigh_servo_attachment_v3.stl; collision mesh filename=package:///9g_servo_arm_v1.stl
- link righthip_2: mass 0.031925376082855685955 -> 0.035352377824358502401; geometry collision mesh filename=package:///18g_thigh_servo_attachment_v3.stl; collision mesh filename=package:///9g_servo_arm_v1.stl
- link rightthigh: mass 0.0018464874791640291558 -> 0.0018464874791640285053
- link rightthigh_2: mass 0.0018464874791640291558 -> 0.0018464874791640285053
Joints:
- removed joint foot_backleft
- removed joint foot_frontleft
- removed joint pivot_backleft
- removed joint pivot_backright
- removed joint pivot_frontleft
- removed joint pivot_frontright
- removed joint thigh_backleft
- removed joint thigh_frontleft
- removed joint topservo_backleft
- removed joint topservo_backright
- removed joint topservo_frontleft
- removed joint topservo_frontright
- added joint femur_backright: type revolute, parent righthip_2, child leftfemur_4, origin xyz=-0.024642932224073363368 -0.019813232385326031565 -0.013275631329225989763 rpy=-1.5707963267948987784 -0.69825389664490622454 1.5707963267948938935, axis 0 0 1, limit effort=1 velocity=20
- added joint femur_frontright: type revolute, parent righthip, child leftfemur_3, origin xyz=-0.024642932224072704173 -0.019813232385325556251 -0.013275631329226038335 rpy=-1.5707963267948990005 -0.68346821395421664125 1.5707963267948936714, axis 0 0 1, limit effort=1 velocity=20
- added joint femur_leftback: type revolute, parent lefthip_2, child leftfemur_2, origin xyz=-0.024650000000000477085 0.019549368670763501293 -0.011775631329240782152 rpy=1.5707963267953368725 -0.67051192598255138222 -1.5707963267951625674, axis 0 0 1, limit effort=1 velocity=20
- added joint femur_leftfront: type revolute, parent lefthip, child leftfemur, origin xyz=-0.024650000000001406897 0.019549368670763487416 -0.011775631329240969503 rpy=1.570796326795334874 -0.66646697390099118863 -1.5707963267951601249, axis 0 0 1, limit effort=1 velocity=20
- added joint foot_leftback: type revolute, parent leftthigh_2, child leftfoot_2, origin xyz=0.035000000000000058842 -2.2759572004815709079e-15 -0.0069999999999998674394 rpy=-3.1415926535897926719 6.6159403471175274119e-15 -1.6625457993150511982, axis 0 0 1, limit lower=0.785398163397448279 upper=1.8325957145940461324 effort=1 velocity=20
- added joint foot_leftfront: type revolute, parent leftthigh, child leftfoot, origin xyz=0.034999999999982094046 -8.0005446712050343194e-15 -0.0069999999999999090727 rpy=-3.1415926535897900074 1.4027236575191825091e-15 -1.6352595016448581156, axis 0 0 1, limit lower=0.785398163397448279 upper=1.8325957145940461324 effort=1 velocity=20
- added joint thigh_leftback: type revolute, parent lefthip_2, child leftthigh_2, origin xyz=-0.017649999999996203448 0.0071749999999998993402 -0.024150000000004223644 rpy=-1.5707963267944760055 -0.64616105155389358394 -1.570796326795150577, axis 0 0 1, limit lower=0.52359877559829881566 upper=1.3089969389957472057 effort=1 velocity=20
- added joint thigh_leftfront: type revolute, parent lefthip, child leftthigh, origin xyz=-0.017649999999996862643 0.0071750000000001751613 -0.024150000000004313849 rpy=-1.5707963267944642372 -0.68299626649609701534 -1.570796326795170117, axis 0 0 1, limit lower=0.52359877559829881566 upper=1.3089969389957472057 effort=1 velocity=20
- joint backlefthip: limit effort=1 velocity=20 -> lower=0 upper=0 effort=1 velocity=20
- joint backrighthip: limit effort=1 velocity=20 -> lower=0 upper=0 effort=1 velocity=20; origin xyz=-0.036799999999999492839 0.15150000000000007905 -7.0476127562967642837e-05 rpy=-1.570796326794896558 0.0069151859789502072642 -1.6654141744842036084e-16 -> xyz=-0.036799999999999492839 0.15150000000000002354 -7.0476127562964105628e-05 rpy=-1.570796326794896336 -4.1633363423443277821e-17 -1.2972374029647262691e-15
- joint foot_backright: limit effort=1 velocity=20 -> lower=2.8797932657906435416 upper=3.926990816987241395 effort=1 velocity=20; origin xyz=0.035000000000003431144 -2.5673907444456744997e-15 -0.0070000000000007209233 rpy=-3.1415926535897624738 -3.8656844969137088255e-14 1.8467252656638426522 -> xyz=0.03499999999999731104 5.273559366969493567e-15 -0.0069999999999999923395 rpy=-3.1415926535897922278 1.278825186765632713e-16 1.605679334027174443
- joint foot_frontright: limit effort=1 velocity=20 -> lower=2.8797932657906435416 upper=3.926990816987241395 effort=1 velocity=20; origin xyz=0.034999999999999975575 -6.5919492087118669588e-17 -0.0069999999999999090727 rpy=3.141592653589793116 1.8112474417422630241e-16 1.7421856465996083951 -> xyz=0.034999999999997137567 -5.089678678515952015e-15 -0.0069999999999990764055 rpy=3.141592653589773132 -3.0284421533315752305e-13 1.5873207190023146396
- joint frontlefthip: limit effort=1 velocity=20 -> lower=0 upper=0 effort=1 velocity=20; origin xyz=0.036800000000000873679 0.056500000000000209777 -0.00047047612756321774679 rpy=1.570796326794896558 -0.034629928912120480633 3.141592653589793116 -> xyz=0.036800000000000845923 0.056500000000000223654 -0.00047047612756321785521 rpy=1.570796326794896558 -1.07552855510556222e-16 3.141592653589793116
- joint frontrighthip: limit effort=1 velocity=20 -> lower=0 upper=0 effort=1 velocity=20; origin xyz=-0.03679999999999954835 0.056500000000000036304 -7.0476127562987795445e-05 rpy=-1.570796326794896558 0.0059585403227931117015 -1.6587782772357954168e-16 -> xyz=-0.036799999999999541411 0.056500000000000057121 -7.047612756298749729e-05 rpy=-1.570796326794896336 -1.732338231197280609e-15 -4.9961410333088865119e-16
- joint thigh_backright: limit effort=1 velocity=20 -> lower=0.52359877559829881566 upper=1.3089969389957472057 effort=1 velocity=20; origin xyz=0 2.2985086056692694001e-17 0 rpy=3.42598261879114307e-16 -8.0380887748982940841e-17 -0.97364841798577050902 -> xyz=-0.017642932224073371028 -0.0074388637145611745394 -0.025649999999990985566 rpy=1.5707963267948943376 -0.68793763179652955841 1.5707963267948961139; parent rightpivot_2 -> righthip_2
- joint thigh_frontright: limit effort=1 velocity=20 -> lower=1.8325957145940461324 upper=2.6179938779914944114 effort=1 velocity=20; origin xyz=-3.4694469519536141888e-18 0 -1.3877787807814456755e-17 rpy=-9.5616091236429676855e-16 -2.5268296817871380792e-17 -0.80308671419846577866 -> xyz=-0.01764293222407292 -0.0074388637145611025484 -0.025649999999990867605 rpy=1.5707963267948941155 -0.72169352917961204774 1.5707963267948936714; parent rightpivot -> righthip

Commit message: movement figured out, ready for RL implementation

File: src/model/robot.urdf (robot description, URDF)
Before this commit: robot onshape, 17 links, 16 joints
Joints:
- joint frontrighthip: limit lower=0 upper=0 effort=1 velocity=20 -> lower=-1.0472 upper=1.0472 effort=100 velocity=100

Commit message: added movement to all joints

File: src/model/robot.urdf (robot description, URDF)
Before this commit: robot onshape, 17 links, 16 joints
Joints:
- joint backlefthip: limit lower=0 upper=0 effort=1 velocity=20 -> lower=-1.0472 upper=1.0472 effort=300 velocity=300
- joint backrighthip: limit lower=0 upper=0 effort=1 velocity=20 -> lower=-1.0472 upper=1.0472 effort=300 velocity=300
- joint femur_backright: limit effort=1 velocity=20 -> effort=300 velocity=300
- joint femur_frontright: limit effort=1 velocity=20 -> effort=300 velocity=300
- joint femur_leftback: limit effort=1 velocity=20 -> effort=300 velocity=300
- joint foot_backright: limit lower=2.8797932657906435416 upper=3.926990816987241395 effort=1 velocity=20 -> lower=2.8797932657906435416 upper=3.926990816987241395 effort=300 velocity=300
- joint foot_frontright: limit lower=2.8797932657906435416 upper=3.926990816987241395 effort=1 velocity=20 -> lower=2.8797932657906435416 upper=3.926990816987241395 effort=300 velocity=300
- joint foot_leftback: limit lower=0.785398163397448279 upper=1.8325957145940461324 effort=1 velocity=20 -> lower=0.785398163397448279 upper=1.8325957145940461324 effort=300 velocity=300
- joint foot_leftfront: limit lower=0.785398163397448279 upper=1.8325957145940461324 effort=1 velocity=20 -> lower=0.785398163397448279 upper=1.8325957145940461324 effort=300 velocity=300
- joint frontlefthip: limit lower=0 upper=0 effort=1 velocity=20 -> lower=-1.0472 upper=1.0472 effort=300 velocity=300
- joint frontrighthip: limit lower=-1.0472 upper=1.0472 effort=100 velocity=100 -> lower=-1.0472 upper=1.0472 effort=300 velocity=300
- joint thigh_backright: limit lower=0.52359877559829881566 upper=1.3089969389957472057 effort=1 velocity=20 -> lower=0.52359877559829881566 upper=1.3089969389957472057 effort=300 velocity=300
- joint thigh_frontright: limit lower=1.8325957145940461324 upper=2.6179938779914944114 effort=1 velocity=20 -> lower=1.8325957145940461324 upper=2.6179938779914944114 effort=300 velocity=300
- joint thigh_leftback: limit lower=0.52359877559829881566 upper=1.3089969389957472057 effort=1 velocity=20 -> lower=0.52359877559829881566 upper=1.3089969389957472057 effort=300 velocity=300
- joint thigh_leftfront: limit lower=0.52359877559829881566 upper=1.3089969389957472057 effort=1 velocity=20 -> lower=0.52359877559829881566 upper=1.3089969389957472057 effort=300 velocity=300

Commit message: fixed limits to be consistent

File: src/model/robot.urdf (robot description, URDF)
Before this commit: robot onshape, 17 links, 16 joints
Joints:
- joint foot_backright: limit lower=2.8797932657906435416 upper=3.926990816987241395 effort=300 velocity=300 -> lower=-1.0472 upper=0 effort=300 velocity=300
- joint foot_frontright: limit lower=2.8797932657906435416 upper=3.926990816987241395 effort=300 velocity=300 -> lower=-1.0472 upper=0 effort=300 velocity=300
- joint foot_leftback: limit lower=0.785398163397448279 upper=1.8325957145940461324 effort=300 velocity=300 -> lower=0 upper=1.0472 effort=300 velocity=300
- joint foot_leftfront: limit lower=0.785398163397448279 upper=1.8325957145940461324 effort=300 velocity=300 -> lower=0 upper=1.0472 effort=300 velocity=300
- joint thigh_backright: limit lower=0.52359877559829881566 upper=1.3089969389957472057 effort=300 velocity=300 -> lower=-1.0472 upper=0 effort=300 velocity=300
- joint thigh_frontright: limit lower=1.8325957145940461324 upper=2.6179938779914944114 effort=300 velocity=300 -> lower=-1.0472 upper=0 effort=300 velocity=300
- joint thigh_leftback: limit lower=0.52359877559829881566 upper=1.3089969389957472057 effort=300 velocity=300 -> lower=0 upper=1.0472 effort=300 velocity=300
- joint thigh_leftfront: limit lower=0.52359877559829881566 upper=1.3089969389957472057 effort=300 velocity=300 -> lower=0 upper=1.0472 effort=300 velocity=300

Commit message: model can successfully move, ready for RL

File: src/model/robot.urdf (robot description, URDF)
Before this commit: robot onshape, 17 links, 16 joints
Joints:
- joint femur_backright: limit effort=300 velocity=300 -> (none); type revolute -> fixed
- joint femur_frontright: limit effort=300 velocity=300 -> (none); type revolute -> fixed
- joint femur_leftback: limit effort=300 velocity=300 -> (none); type revolute -> fixed
- joint femur_leftfront: limit effort=1 velocity=20 -> (none); type revolute -> fixed
