Commit message: stuck on first step

File: src/robot/robot.urdf (robot description, URDF)
Before this commit: robot onshape, 17 links, 16 joints
Links:
- link chassis: mass 0.14444259148618379673 -> 0.33140859148618373453; geometry collision mesh filename=package:///18g_servo_v1.stl; collision mesh filename=package:///18g_servo_v1.stl
- link lefthip: mass 0.035898853366757597916 -> 0.035898853366757604855
- link leftthigh: mass 0.0018464875329195404828 -> 0.0018464875329195406996
- link leftthigh_2: mass 0.0018464875329195404828 -> 0.0018464875329195406996
- link rightfoot: mass 0.0052504289083666246668 -> 0.0052504289083666264015
- link rightfoot_2: mass 0.0052504289083666246668 -> 0.0052504289083666264015
- link rightthigh: mass 0.0018464874791640285053 -> 0.0018464874791640291558
- link rightthigh_2: mass 0.0018464874791640285053 -> 0.0018464874791640291558
Joints:
- joint backlefthip: limit lower=-1.0472 upper=1.0472 effort=300 velocity=300 -> lower=-0.261799 upper=0.261799 effort=1 velocity=20; origin xyz=0.036800000000000568368 0.15150000000000005129 -0.00047047612756297499392 rpy=1.570796326794896558 -1.0648674274956604569e-16 3.141592653589793116 -> xyz=0.036800000000000526734 0.15150000000000207745 -0.00047047612756298231229 rpy=1.570796326794896558 -1.0648674274956321072e-16 -3.141592653589783346
- joint backrighthip: limit lower=-1.0472 upper=1.0472 effort=300 velocity=300 -> lower=-0.261799 upper=0.261799 effort=1 velocity=20; origin xyz=-0.036799999999999492839 0.15150000000000002354 -7.0476127562964105628e-05 rpy=-1.570796326794896336 -4.1633363423443277821e-17 -1.2972374029647262691e-15 -> xyz=-0.036800000000002490441 0.15150000000000204969 -7.0476127562969092958e-05 rpy=-1.570796326794896558 1.0648674274956146044e-16 7.5640658693905968835e-15
- joint femur_backright: limit (none) -> effort=1 velocity=20; origin xyz=-0.024642932224073363368 -0.019813232385326031565 -0.013275631329225989763 rpy=-1.5707963267948987784 -0.69825389664490622454 1.5707963267948938935 -> xyz=-0.024642932224073370306 -0.019813232385326069729 -0.013275631329226017519 rpy=-1.5707963267948983344 -0.69825389664490655761 1.5707963267948947816; type fixed -> revolute
- joint femur_frontright: limit (none) -> effort=1 velocity=20; origin xyz=-0.024642932224072704173 -0.019813232385325556251 -0.013275631329226038335 rpy=-1.5707963267948990005 -0.68346821395421664125 1.5707963267948936714 -> xyz=-0.024642932224072711112 -0.019813232385325504209 -0.013275631329226003641 rpy=-1.5707963267948983344 -0.68346821395421686329 1.570796326794891673; type fixed -> revolute
- joint femur_leftback: limit (none) -> effort=1 velocity=20; origin xyz=-0.024650000000000477085 0.019549368670763501293 -0.011775631329240782152 rpy=1.5707963267953368725 -0.67051192598255138222 -1.5707963267951625674 -> xyz=-0.024650000000000588107 0.019549368670763497824 -0.011775631329240782152 rpy=1.5707963267953368725 -0.67051192598255138222 -1.5707963267951625674; type fixed -> revolute
- joint femur_leftfront: limit (none) -> effort=1 velocity=20; origin xyz=-0.024650000000001406897 0.019549368670763487416 -0.011775631329240969503 rpy=1.570796326795334874 -0.66646697390099118863 -1.5707963267951601249 -> xyz=-0.024650000000001379141 0.019549368670763494354 -0.011775631329240955625 rpy=1.5707963267953350961 -0.66646697390099118863 -1.5707963267951601249; type fixed -> revolute
- joint foot_backright: limit lower=-1.0472 upper=0 effort=300 velocity=300 -> lower=-1.0472 upper=0 effort=1 velocity=20; origin xyz=0.03499999999999731104 5.273559366969493567e-15 -0.0069999999999999923395 rpy=-3.1415926535897922278 1.278825186765632713e-16 1.605679334027174443 -> xyz=0.034999999999997297162 5.2458037913538646535e-15 -0.0069999999999999923395 rpy=-3.141592653589793116 2.2441480830048960661e-16 1.4414733445528478128
- joint foot_frontright: limit lower=-1.0472 upper=0 effort=300 velocity=300 -> lower=-1.0472 upper=0 effort=1 velocity=20; origin xyz=0.034999999999997137567 -5.089678678515952015e-15 -0.0069999999999990764055 rpy=3.141592653589773132 -3.0284421533315752305e-13 1.5873207190023146396 -> xyz=0.034999999999991295019 -3.3098523921637479361e-15 -0.0069999999999990347721 rpy=3.141592653589793116 5.3157713190766779058e-16 1.773434614324501446
- joint foot_leftback: limit lower=0 upper=1.0472 effort=300 velocity=300 -> lower=0 upper=1.0472 effort=1 velocity=20; origin xyz=0.035000000000000058842 -2.2759572004815709079e-15 -0.0069999999999998674394 rpy=-3.1415926535897926719 6.6159403471175274119e-15 -1.6625457993150511982 -> xyz=0.035000000000000114353 -2.4286128663675299322e-15 -0.0069999999999998813172 rpy=-3.1415926535897926719 6.666559147123260302e-15 -1.6625457993150511982
- joint foot_leftfront: limit lower=0 upper=1.0472 effort=300 velocity=300 -> lower=0 upper=1.0472 effort=1 velocity=20; origin xyz=0.034999999999982094046 -8.0005446712050343194e-15 -0.0069999999999999090727 rpy=-3.1415926535897900074 1.4027236575191825091e-15 -1.6352595016448581156 -> xyz=0.034999999999982038534 -7.9831974364452662485e-15 -0.0069999999999999090727 rpy=-3.1415926535897900074 1.5819249601435661476e-15 -1.6352595016448581156
- joint frontlefthip: limit lower=-1.0472 upper=1.0472 effort=300 velocity=300 -> lower=-0.261799 upper=0.261799 effort=1 velocity=20; origin xyz=0.036800000000000845923 0.056500000000000223654 -0.00047047612756321785521 rpy=1.570796326794896558 -1.07552855510556222e-16 3.141592653589793116 -> xyz=0.036800000000001262257 0.05650000000000113265 -0.00047047612756291601332 rpy=1.570796326794896558 -1.0668549377256967968e-16 -3.141592653589788231
- joint frontrighthip: limit lower=-1.0472 upper=1.0472 effort=300 velocity=300 -> lower=-0.261799 upper=0.261799 effort=1 velocity=20; origin xyz=-0.036799999999999541411 0.056500000000000057121 -7.047612756298749729e-05 rpy=-1.570796326794896336 -1.732338231197280609e-15 -4.9961410333088865119e-16 -> xyz=-0.036800000000001581446 0.056500000000000778766 -7.0476127562992511725e-05 rpy=-1.570796326794896558 -1.7106901340672024212e-16 9.1593124686582624559e-15
- joint thigh_backright: limit lower=-1.0472 upper=0 effort=300 velocity=300 -> lower=-1.0472 upper=0 effort=1 velocity=20; origin xyz=-0.017642932224073371028 -0.0074388637145611745394 -0.025649999999990985566 rpy=1.5707963267948943376 -0.68793763179652955841 1.5707963267948961139 -> xyz=-0.017642932224073377967 -0.0074388637145611710699 -0.025649999999990985566 rpy=1.5707963267948950037 -0.76963751995166607145 1.5707963267948952257
- joint thigh_frontright: limit lower=-1.0472 upper=0 effort=300 velocity=300 -> lower=-1.0472 upper=0 effort=1 velocity=20; origin xyz=-0.01764293222407292 -0.0074388637145611025484 -0.025649999999990867605 rpy=1.5707963267948941155 -0.72169352917961204774 1.5707963267948936714 -> xyz=-0.017642932224072947756 -0.0074388637145610548435 -0.025649999999990853727 rpy=1.5707963267948954478 -0.63152345479824956165 1.5707963267948918951
- joint thigh_leftback: limit lower=0 upper=1.0472 effort=300 velocity=300 -> lower=0 upper=1.0472 effort=1 velocity=20; origin xyz=-0.017649999999996203448 0.0071749999999998993402 -0.024150000000004223644 rpy=-1.5707963267944760055 -0.64616105155389358394 -1.570796326795150577 -> xyz=-0.017649999999996203448 0.0071749999999998993402 -0.024150000000004251399 rpy=-1.5707963267948976682 -0.64616105155389358394 -1.5707963267948978903
- joint thigh_leftfront: limit lower=0 upper=1.0472 effort=300 velocity=300 -> lower=0 upper=1.0472 effort=1 velocity=20; origin xyz=-0.017649999999996862643 0.0071750000000001751613 -0.024150000000004313849 rpy=-1.5707963267944642372 -0.68299626649609701534 -1.570796326795170117 -> xyz=-0.017649999999997466327 0.0071749999999998707173 -0.024150000000004362422 rpy=-1.5707963267949041075 -0.68299626649609701534 -1.5707963267948936714

Commit message: changed robot, changed implementation of action space

File: src/robot/robot.urdf (robot description, URDF)
Before this commit: robot onshape, 17 links, 16 joints
Links:
- removed link leftfemur
- removed link leftfemur_2
- removed link leftfemur_3
- removed link leftfemur_4
- link chassis: mass 0.33140859148618373453 -> 0.31717023469841981731; geometry collision mesh filename=package:///18g_servo_v1.stl; collision mesh filename=package:///18g_servo_v1.stl
- link leftfoot: mass 0.0052313671076180037062 -> 0.0050411870565304911507
- link leftfoot_2: mass 0.0052313671076180037062 -> 0.0050411870565304911507
- link leftthigh: mass 0.0018464875329195406996 -> 0.0018464875329195404828
- link leftthigh_2: mass 0.0018464875329195406996 -> 0.0018464875329195404828
- link rightfoot: mass 0.0052504289083666264015 -> 0.005060248979884990686
- link rightfoot_2: mass 0.0052504289083666264015 -> 0.005060248979884990686
- link rightthigh: mass 0.0018464874791640291558 -> 0.0018464874791640287222
- link rightthigh_2: mass 0.0018464874791640291558 -> 0.0018464874791640287222
Joints:
- removed joint femur_backright
- removed joint femur_frontright
- removed joint femur_leftback
- removed joint femur_leftfront
- joint foot_frontright: origin xyz=0.034999999999991295019 -3.3098523921637479361e-15 -0.0069999999999990347721 rpy=3.141592653589793116 5.3157713190766779058e-16 1.773434614324501446 -> xyz=0.034999999999991301958 -3.2959746043559334794e-15 -0.0069999999999990278332 rpy=-3.141592653589793116 5.6029632860372716604e-16 1.7734346143245007799
- joint foot_leftback: origin xyz=0.035000000000000114353 -2.4286128663675299322e-15 -0.0069999999999998813172 rpy=-3.1415926535897926719 6.666559147123260302e-15 -1.6625457993150511982 -> xyz=0.035000000000000114353 -2.4147350785597154754e-15 -0.0069999999999998813172 rpy=-3.1415926535897926719 6.6665591471232595132e-15 -1.6625457993150511982
- joint foot_leftfront: origin xyz=0.034999999999982038534 -7.9831974364452662485e-15 -0.0069999999999999090727 rpy=-3.1415926535897900074 1.5819249601435661476e-15 -1.6352595016448581156 -> xyz=0.034999999999982045473 -7.9831974364452662485e-15 -0.0069999999999999090727 rpy=-3.1415926535897900074 1.5819249601435221686e-15 -1.6352595016448581156
- joint frontlefthip: origin xyz=0.036800000000001262257 0.05650000000000113265 -0.00047047612756291601332 rpy=1.570796326794896558 -1.0668549377256967968e-16 -3.141592653589788231 -> xyz=0.036800000000000311629 0.056500000000000973055 -0.00047047612756290647235 rpy=1.570796326794896558 -1.064867427495631984e-16 3.141592653589793116
- joint thigh_frontright: origin xyz=-0.017642932224072947756 -0.0074388637145610548435 -0.025649999999990853727 rpy=1.5707963267948954478 -0.63152345479824956165 1.5707963267948918951 -> xyz=-0.017642932224073031022 -0.0074388637145610652518 -0.025649999999990871075 rpy=1.5707963267948956698 -0.63152345479825011676 1.570796326794891673
- joint thigh_leftback: origin xyz=-0.017649999999996203448 0.0071749999999998993402 -0.024150000000004251399 rpy=-1.5707963267948976682 -0.64616105155389358394 -1.5707963267948978903 -> xyz=-0.017649999999996210387 0.0071749999999999028097 -0.024150000000004334666 rpy=-1.5707963267948976682 -0.64616105155389358394 -1.5707963267948978903
- joint thigh_leftfront: origin xyz=-0.017649999999997466327 0.0071749999999998707173 -0.024150000000004362422 rpy=-1.5707963267949041075 -0.68299626649609701534 -1.5707963267948936714 -> xyz=-0.017649999999996862643 0.0071750000000001812328 -0.024150000000004272216 rpy=-1.5707963267949105468 -0.68299626649609701534 -1.5707963267948894526

Commit message: Addded tips and continued training modifications

File: src/robot/robot.urdf (robot description, URDF)
Before this commit: robot onshape, 13 links, 12 joints
Links:
- added link part_1, mass 0; collision mesh filename=package:///part_1.stl; visual mesh filename=package:///part_1.stl
- added link part_1_2, mass 0; collision mesh filename=package:///part_1.stl; visual mesh filename=package:///part_1.stl
- added link part_1_3, mass 0; collision mesh filename=package:///part_1.stl; visual mesh filename=package:///part_1.stl
- added link part_1_4, mass 0; collision mesh filename=package:///part_1.stl; visual mesh filename=package:///part_1.stl
- link chassis: mass 0.31717023469841981731 -> 0.31717023469841987282
- link leftfoot: mass 0.0050411870565304911507 -> 0.0050411870565304902833
- link leftfoot_2: mass 0.0050411870565304911507 -> 0.0050411870565304902833
- link righthip: mass 0.035352377824358502401 -> 0.035352377824358509339
- link righthip_2: mass 0.035352377824358502401 -> 0.035352377824358509339
Joints:
- added joint backlefttip: type revolute, parent leftfoot_2, child part_1_2, origin xyz=-0.039415880433163880125 -0.002549509756796353166 -0.0012499999999999941713 rpy=-2.6179938779914930791 -1.570796326794896558 0, axis 0 0 1, limit effort=1 velocity=20
- added joint backrighttip: type revolute, parent rightfoot_2, child part_1_4, origin xyz=-0.039415880433163887064 0.0025495097567963670437 -0.0012500000000000011102 rpy=0.52359877559829925975 1.570796326794896558 0, axis 0 0 1, limit effort=1 velocity=20
- added joint frontlefttip: type revolute, parent leftfoot, child part_1, origin xyz=-0.039415880433163956453 -0.0025495097567964086771 -0.0012499999999999941713 rpy=-2.6179938779914930791 -1.570796326794896558 0, axis 0 0 1, limit effort=1 velocity=20
- added joint frontrighttip: type revolute, parent rightfoot, child part_1_3, origin xyz=-0.039415880433163935637 0.0025495097567963878604 -0.0012500000000000011102 rpy=0.52359877559829914873 1.570796326794896558 0, axis 0 0 1, limit effort=1 velocity=20
- joint foot_backright: origin xyz=0.034999999999997297162 5.2458037913538646535e-15 -0.0069999999999999923395 rpy=-3.141592653589793116 2.2441480830048960661e-16 1.4414733445528478128 -> xyz=0.034999999999997172262 5.0515147620444622589e-15 -0.0070000000000000062172 rpy=-3.1415926535897922278 1.2935959933079770153e-16 1.6042252411713742166
- joint foot_leftback: origin xyz=0.035000000000000114353 -2.4147350785597154754e-15 -0.0069999999999998813172 rpy=-3.1415926535897926719 6.6665591471232595132e-15 -1.6625457993150511982 -> xyz=0.035000000000000100475 -2.4147350785597154754e-15 -0.0069999999999998882561 rpy=-3.1415926535897926719 6.6665591471232532023e-15 -1.6625457993150511982
- joint foot_leftfront: origin xyz=0.034999999999982045473 -7.9831974364452662485e-15 -0.0069999999999999090727 rpy=-3.1415926535897900074 1.5819249601435221686e-15 -1.6352595016448581156 -> xyz=0.034999999999982045473 -7.9831974364452662485e-15 -0.0069999999999999160116 rpy=-3.1415926535897900074 1.5819249601435221686e-15 -1.6352595016448581156
- joint thigh_backright: origin xyz=-0.017642932224073377967 -0.0074388637145611710699 -0.025649999999990985566 rpy=1.5707963267948950037 -0.76963751995166607145 1.5707963267948952257 -> xyz=-0.017642932224073391845 -0.0074388637145611710699 -0.025649999999990846788 rpy=1.5707963267948947816 -0.69429000070910196207 1.5707963267948956698
- joint thigh_leftback: origin xyz=-0.017649999999996210387 0.0071749999999999028097 -0.024150000000004334666 rpy=-1.5707963267948976682 -0.64616105155389358394 -1.5707963267948978903 -> xyz=-0.017649999999996210387 0.0071749999999999028097 -0.024150000000004334666 rpy=-1.5707963267948981123 -0.64616105155389358394 -1.5707963267948972241
- joint thigh_leftfront: origin xyz=-0.017649999999996862643 0.0071750000000001812328 -0.024150000000004272216 rpy=-1.5707963267949105468 -0.68299626649609701534 -1.5707963267948894526 -> xyz=-0.017649999999996855704 0.0071750000000001829675 -0.024150000000004272216 rpy=-1.5707963267949105468 -0.68299626649609701534 -1.5707963267948894526
